Commit message: updates on controller

File: urdf/agent.urdf (robot description, URDF)
Before this commit: robot agent, 9 links, 8 joints
Links:
- link agent: geometry collision mesh filename=package://home/nidhi/reactive_nav/model/cube.obj scale=1. 1. 1.; visual mesh filename=package://home/nidhi/reactive_nav/model/cube.obj scale=1. 1. 1.
- link base: geometry collision mesh filename=package://home/nidhi/reactive_nav/model/cube.obj scale=10 10 .01; visual mesh filename=package://home/nidhi/reactive_nav/model/cube.obj scale=10 10 .01
- link base_wall1: geometry collision mesh filename=package://home/nidhi/reactive_nav/model/cube.obj scale=10 .01 5; visual mesh filename=package://home/nidhi/reactive_nav/model/cube.obj scale=10 .01 5
- link base_wall2: geometry collision mesh filename=package://home/nidhi/reactive_nav/model/cube.obj scale=10 .01 5; visual mesh filename=package://home/nidhi/reactive_nav/model/cube.obj scale=10 .01 5
- link base_wall3: geometry collision mesh filename=package://home/nidhi/reactive_nav/model/cube.obj scale=0.01 10 5; visual mesh filename=package://home/nidhi/reactive_nav/model/cube.obj scale=.01 10 5
- link base_wall4: geometry collision mesh filename=package://home/nidhi/reactive_nav/model/cube.obj scale=0.01 10 5; visual mesh filename=package://home/nidhi/reactive_nav/model/cube.obj scale=.01 10 5
- link obstacle: geometry collision mesh filename=package://home/nidhi/reactive_nav/model/cube.obj scale=1 1 1.5; visual mesh filename=package://home/nidhi/reactive_nav/model/cube.obj scale=1 1 1.5

Commit message: completed force and postion coupled controller

File: urdf/agent.urdf (robot description, URDF)
Before this commit: robot agent, 9 links, 8 joints
Links:
- link obstacle: mass None -> 10
Joints:
- joint joint2: limit lower=-15 upper=5 effort=1000.0 velocity=.1 -> lower=-15 upper=5 effort=100000.0 velocity=.1
- joint world_ob: limit lower=-.01 upper=1 effort=1000.0 velocity=.1 -> lower=0 upper=.01 effort=.0001 velocity=.1
